Commit message: Release v1.0.2

File: fanuc_crx_description/urdf/crx10ia_l_urdf_macro.xacro (robot description, xacro)
@@ -6,7 +6,4 @@
 -->
 <robot xmlns:xacro="http://wiki.ros.org/xacro">
-  <xacro:include
-    filename="$(find fanuc_crx_description)/urdf/fanuc_common_urdf_macro.xacro"
-  />
   <xacro:macro
     name="crx10ia_l"
@@ -62,5 +59,4 @@
           />
         </geometry>
-        <material name="FANUC_Black" />
       </visual>
       <collision>
@@ -94,5 +90,4 @@
           />
         </geometry>
-        <material name="FANUC_White" />
       </visual>
       <collision>
@@ -126,5 +121,4 @@
           />
         </geometry>
-        <material name="FANUC_White" />
       </visual>
       <collision>
@@ -158,5 +152,4 @@
           />
         </geometry>
-        <material name="FANUC_White" />
       </visual>
       <collision>
@@ -190,5 +183,4 @@
           />
         </geometry>
-        <material name="FANUC_White" />
       </visual>
       <collision>
@@ -225,5 +217,4 @@
           />
         </geometry>
-        <material name="FANUC_White" />
       </visual>
       <collision>
@@ -260,5 +251,4 @@
           />
         </geometry>
-        <material name="FANUC_Black" />
       </visual>
       <collision>

File: fanuc_crx_description/urdf/crx10ia_urdf_macro.xacro (robot description, xacro)
@@ -6,7 +6,4 @@
 -->
 <robot xmlns:xacro="http://wiki.ros.org/xacro">
-  <xacro:include
-    filename="$(find fanuc_crx_description)/urdf/fanuc_common_urdf_macro.xacro"
-  />
   <xacro:macro
     name="crx10ia"
@@ -62,5 +59,4 @@
           />
         </geometry>
-        <material name="FANUC_Black" />
       </visual>
       <collision>
@@ -94,5 +90,4 @@
           />
         </geometry>
-        <material name="FANUC_White" />
       </visual>
       <collision>
@@ -126,5 +121,4 @@
           />
         </geometry>
-        <material name="FANUC_White" />
       </visual>
       <collision>
@@ -158,5 +152,4 @@
           />
         </geometry>
-        <material name="FANUC_White" />
       </visual>
       <collision>
@@ -190,5 +183,4 @@
           />
         </geometry>
-        <material name="FANUC_White" />
       </visual>
       <collision>
@@ -225,5 +217,4 @@
           />
         </geometry>
-        <material name="FANUC_White" />
       </visual>
       <collision>
@@ -260,5 +251,4 @@
           />
         </geometry>
-        <material name="FANUC_Black" />
       </visual>
       <collision>

File: fanuc_crx_description/urdf/crx20ia_l_urdf_macro.xacro (robot description, xacro)
@@ -6,7 +6,4 @@
 -->
 <robot xmlns:xacro="http://wiki.ros.org/xacro">
-  <xacro:include
-    filename="$(find fanuc_crx_description)/urdf/fanuc_common_urdf_macro.xacro"
-  />
   <xacro:macro
     name="crx20ia_l"
@@ -62,5 +59,4 @@
           />
         </geometry>
-        <material name="FANUC_Black" />
       </visual>
       <collision>
@@ -94,5 +90,4 @@
           />
         </geometry>
-        <material name="FANUC_White" />
       </visual>
       <collision>
@@ -126,5 +121,4 @@
           />
         </geometry>
-        <material name="FANUC_White" />
       </visual>
       <collision>
@@ -158,5 +152,4 @@
           />
         </geometry>
-        <material name="FANUC_White" />
       </visual>
       <collision>
@@ -190,5 +183,4 @@
           />
         </geometry>
-        <material name="FANUC_White" />
       </visual>
       <collision>
@@ -225,5 +217,4 @@
           />
         </geometry>
-        <material name="FANUC_White" />
       </visual>
       <collision>
@@ -260,5 +251,4 @@
           />
         </geometry>
-        <material name="FANUC_Black" />
       </visual>
       <collision>

File: fanuc_crx_description/urdf/crx30ia_urdf_macro.xacro (robot description, xacro)
@@ -6,7 +6,4 @@
 -->
 <robot xmlns:xacro="http://wiki.ros.org/xacro">
-  <xacro:include
-    filename="$(find fanuc_crx_description)/urdf/fanuc_common_urdf_macro.xacro"
-  />
   <xacro:macro
     name="crx30ia"
@@ -62,5 +59,4 @@
           />
         </geometry>
-        <material name="FANUC_Black" />
       </visual>
       <collision>
@@ -94,5 +90,4 @@
           />
         </geometry>
-        <material name="FANUC_White" />
       </visual>
       <collision>
@@ -126,5 +121,4 @@
           />
         </geometry>
-        <material name="FANUC_White" />
       </visual>
       <collision>
@@ -158,5 +152,4 @@
           />
         </geometry>
-        <material name="FANUC_White" />
       </visual>
       <collision>
@@ -190,5 +183,4 @@
           />
         </geometry>
-        <material name="FANUC_White" />
       </visual>
       <collision>
@@ -222,5 +214,4 @@
           />
         </geometry>
-        <material name="FANUC_White" />
       </visual>
       <collision>
@@ -254,5 +245,4 @@
           />
         </geometry>
-        <material name="FANUC_Black" />
       </visual>
       <collision>

File: fanuc_crx_description/urdf/crx5ia_urdf_macro.xacro (robot description, xacro)
@@ -6,7 +6,4 @@
 -->
 <robot xmlns:xacro="http://wiki.ros.org/xacro">
-  <xacro:include
-    filename="$(find fanuc_crx_description)/urdf/fanuc_common_urdf_macro.xacro"
-  />
   <xacro:macro
     name="crx5ia"
@@ -62,5 +59,4 @@
           />
         </geometry>
-        <material name="FANUC_Black" />
       </visual>
       <collision>
@@ -94,5 +90,4 @@
           />
         </geometry>
-        <material name="FANUC_White" />
       </visual>
       <collision>
@@ -126,5 +121,4 @@
           />
         </geometry>
-        <material name="FANUC_White" />
       </visual>
       <collision>
@@ -158,5 +152,4 @@
           />
         </geometry>
-        <material name="FANUC_White" />
       </visual>
       <collision>
@@ -190,5 +183,4 @@
           />
         </geometry>
-        <material name="FANUC_White" />
       </visual>
       <collision>
@@ -222,5 +214,4 @@
           />
         </geometry>
-        <material name="FANUC_White" />
       </visual>
       <collision>
@@ -257,5 +248,4 @@
           />
         </geometry>
-        <material name="FANUC_Black" />
       </visual>
       <collision>
