Commit message: Release v1.2.0

File: fanuc_r1000ia_description/urdf/r1000ia_100f_urdf_macro.xacro (robot description, xacro)
@@ -1,9 +1,9 @@
 <?xml version="1.0" ?>
 <!--
-SPDX-FileCopyrightText: 2025, FANUC America Corporation
-SPDX-FileCopyrightText: 2025, FANUC CORPORATION
+SPDX-FileCopyrightText: 2025-2026, FANUC America Corporation
+SPDX-FileCopyrightText: 2025-2026, FANUC CORPORATION
 SPDX-License-Identifier: Apache-2.0
 -->
-<!-- URDF for R-1000/100-22A(R-1000iA/100F) -->
+<!-- URDF for R-1000/100F-22A(R-1000iA/100F) -->
 <robot xmlns:xacro="http://wiki.ros.org/xacro">
   <xacro:macro
@@ -20,22 +20,22 @@
     <xacro:property name="j5_lower_limit" value="${radians(-125)}" />
     <xacro:property name="j6_lower_limit" value="${radians(-360)}" />
-    <xacro:property name="j1_upper_limit" value="${radians( 180)}" />
-    <xacro:property name="j2_upper_limit" value="${radians( 155)}" />
-    <xacro:property name="j3_upper_limit" value="${radians( 140)}" />
-    <xacro:property name="j4_upper_limit" value="${radians( 360)}" />
-    <xacro:property name="j5_upper_limit" value="${radians( 125)}" />
-    <xacro:property name="j6_upper_limit" value="${radians( 360)}" />
-    <xacro:property name="j1_effort_limit" value="0" />
-    <xacro:property name="j2_effort_limit" value="0" />
-    <xacro:property name="j3_effort_limit" value="0" />
-    <xacro:property name="j4_effort_limit" value="0" />
-    <xacro:property name="j5_effort_limit" value="0" />
-    <xacro:property name="j6_effort_limit" value="0" />
-    <xacro:property name="j1_velocity_limit" value="${radians( 130)}" />
-    <xacro:property name="j2_velocity_limit" value="${radians( 110)}" />
-    <xacro:property name="j3_velocity_limit" value="${radians( 120)}" />
-    <xacro:property name="j4_velocity_limit" value="${radians( 170)}" />
-    <xacro:property name="j5_velocity_limit" value="${radians( 170)}" />
-    <xacro:property name="j6_velocity_limit" value="${radians( 250)}" />
+    <xacro:property name="j1_upper_limit" value="${radians(180)}" />
+    <xacro:property name="j2_upper_limit" value="${radians(155)}" />
+    <xacro:property name="j3_upper_limit" value="${radians(140)}" />
+    <xacro:property name="j4_upper_limit" value="${radians(360)}" />
+    <xacro:property name="j5_upper_limit" value="${radians(125)}" />
+    <xacro:property name="j6_upper_limit" value="${radians(360)}" />
+    <xacro:property name="j1_effort_limit" value="9000" />
+    <xacro:property name="j2_effort_limit" value="20000" />
+    <xacro:property name="j3_effort_limit" value="8000" />
+    <xacro:property name="j4_effort_limit" value="3000" />
+    <xacro:property name="j5_effort_limit" value="3000" />
+    <xacro:property name="j6_effort_limit" value="2000" />
+    <xacro:property name="j1_velocity_limit" value="${radians(130)}" />
+    <xacro:property name="j2_velocity_limit" value="${radians(110)}" />
+    <xacro:property name="j3_velocity_limit" value="${radians(120)}" />
+    <xacro:property name="j4_velocity_limit" value="${radians(170)}" />
+    <xacro:property name="j5_velocity_limit" value="${radians(170)}" />
+    <xacro:property name="j6_velocity_limit" value="${radians(250)}" />
     <!-- links -->
     <link name="${prefix}base_link">
@@ -53,8 +53,19 @@
           <mesh
             filename="package://fanuc_r1000ia_description/meshes/r1000ia_100f/collision/base.stl"
-            scale="0.001 0.001 0.001"
-          />
-        </geometry>
-      </collision>
+          />
+        </geometry>
+      </collision>
+      <inertial>
+        <mass value=" 137" />
+        <origin xyz="-.129  .0048  .117" />
+        <inertia
+          ixx=" 2.71"
+          ixy=" .241"
+          ixz="-.158"
+          iyy=" 6.08"
+          iyz=" .015"
+          izz=" 7.49"
+        />
+      </inertial>
     </link>
     <link name="${prefix}J1_link">
@@ -72,8 +83,19 @@
           <mesh
             filename="package://fanuc_r1000ia_description/meshes/r1000ia_100f/collision/j1.stl"
-            scale="0.001 0.001 0.001"
-          />
-        </geometry>
-      </collision>
+          />
+        </geometry>
+      </collision>
+      <inertial>
+        <mass value=" 185" />
+        <origin xyz=" .133 -.00239 -.0395" />
+        <inertia
+          ixx=" 4.93"
+          ixy="-.262"
+          ixz="-.216"
+          iyy=" 7.33"
+          iyz=" .424"
+          izz=" 7.6"
+        />
+      </inertial>
     </link>
     <link name="${prefix}J2_link">
@@ -91,8 +113,19 @@
           <mesh
             filename="package://fanuc_r1000ia_description/meshes/r1000ia_100f/collision/j2.stl"
-            scale="0.001 0.001 0.001"
-          />
-        </geometry>
-      </collision>
+          />
+        </geometry>
+      </collision>
+      <inertial>
+        <mass value=" 111" />
+        <origin xyz=" .00598  .148  .394" />
+        <inertia
+          ixx=" 10.5"
+          ixy="-.00257"
+          ixz=" .00636"
+          iyy=" 10.9"
+          iyz="-.17"
+          izz=" 1.04"
+        />
+      </inertial>
     </link>
     <link name="${prefix}J3_link">
@@ -110,8 +143,19 @@
           <mesh
             filename="package://fanuc_r1000ia_description/meshes/r1000ia_100f/collision/j3.stl"
-            scale="0.001 0.001 0.001"
-          />
-        </geometry>
-      </collision>
+          />
+        </geometry>
+      </collision>
+      <inertial>
+        <mass value=" 208" />
+        <origin xyz=" .238  .011  .139" />
+        <inertia
+          ixx=" 5.25"
+          ixy="-.0585"
+          ixz="-1.92"
+          iyy=" 13.4"
+          iyz="-.209"
+          izz=" 12.6"
+        />
+      </inertial>
     </link>
     <link name="${prefix}J4_link">
@@ -129,8 +173,19 @@
           <mesh
             filename="package://fanuc_r1000ia_description/meshes/r1000ia_100f/collision/j4.stl"
-            scale="0.001 0.001 0.001"
-          />
-        </geometry>
-      </collision>
+          />
+        </geometry>
+      </collision>
+      <inertial>
+        <mass value=" 7.97" />
+        <origin xyz=" .929 -.00482  1.99E-16" />
+        <inertia
+          ixx=" .0233"
+          ixy=" .00217"
+          ixz=" 3.02E-15"
+          iyy=" .0512"
+          iyz=" .00000000000462"
+          izz=" .0487"
+        />
+      </inertial>
     </link>
     <link name="${prefix}J5_link">
@@ -148,8 +203,19 @@
           <mesh
             filename="package://fanuc_r1000ia_description/meshes/r1000ia_100f/collision/j5.stl"
-            scale="0.001 0.001 0.001"
-          />
-        </geometry>
-      </collision>
+          />
+        </geometry>
+      </collision>
+      <inertial>
+        <mass value=" 15.5" />
+        <origin xyz=" .0473 -.0132 -.00000000107" />
+        <inertia
+          ixx=" .0866"
+          ixy="-.012"
+          ixz="-.000000000378"
+          iyy=" .107"
+          iyz="-.00000000097"
+          izz=" .13"
+        />
+      </inertial>
     </link>
     <link name="${prefix}J6_link">
@@ -167,8 +233,19 @@
           <mesh
             filename="package://fanuc_r1000ia_description/meshes/r1000ia_100f/collision/j6.stl"
-            scale="0.001 0.001 0.001"
-          />
-        </geometry>
-      </collision>
+          />
+        </geometry>
+      </collision>
+      <inertial>
+        <mass value=" .431" />
+        <origin xyz=" .181  .000127  .000171" />
+        <inertia
+          ixx=" .000858"
+          ixy="-.00000000000219"
+          ixz="-.000000468"
+          iyy=" .000438"
+          iyz=" .0000000000661"
+          izz=" .000443"
+        />
+      </inertial>
     </link>
     <!-- joints -->
@@ -259,4 +336,11 @@
       <child link="${prefix}flange" />
     </joint>
+    <!-- FANUC flange coords -->
+    <link name="${prefix}fanuc_flange" />
+    <joint name="${prefix}flange-fanuc_flange" type="fixed">
+      <origin xyz="0 0 0" rpy="${radians( 180)} ${radians(-90)} ${radians( 0)}" />
+      <parent link="${prefix}flange" />
+      <child link="${prefix}fanuc_flange" />
+    </joint>
     <!-- Attach to parent -->
     <joint name="${prefix}base_joint" type="fixed">

File: fanuc_r2000_description/urdf/r2000ic_125l_urdf_macro.xacro (robot description, xacro)
@@ -1,6 +1,6 @@
 <?xml version="1.0" ?>
 <!--
-SPDX-FileCopyrightText: 2025, FANUC America Corporation
-SPDX-FileCopyrightText: 2025, FANUC CORPORATION
+SPDX-FileCopyrightText: 2025-2026, FANUC America Corporation
+SPDX-FileCopyrightText: 2025-2026, FANUC CORPORATION
 SPDX-License-Identifier: Apache-2.0
 -->
@@ -20,22 +20,22 @@
     <xacro:property name="j5_lower_limit" value="${radians(-125)}" />
     <xacro:property name="j6_lower_limit" value="${radians(-360)}" />
-    <xacro:property name="j1_upper_limit" value="${radians( 185)}" />
-    <xacro:property name="j2_upper_limit" value="${radians( 76)}" />
-    <xacro:property name="j3_upper_limit" value="${radians( 180)}" />
-    <xacro:property name="j4_upper_limit" value="${radians( 360)}" />
-    <xacro:property name="j5_upper_limit" value="${radians( 125)}" />
-    <xacro:property name="j6_upper_limit" value="${radians( 360)}" />
-    <xacro:property name="j1_effort_limit" value=" 10000" />
-    <xacro:property name="j2_effort_limit" value=" 20000" />
-    <xacro:property name="j3_effort_limit" value=" 10000" />
-    <xacro:property name="j4_effort_limit" value=" 4000" />
-    <xacro:property name="j5_effort_limit" value=" 4000" />
-    <xacro:property name="j6_effort_limit" value=" 2000" />
-    <xacro:property name="j1_velocity_limit" value="${radians( 130)}" />
-    <xacro:property name="j2_velocity_limit" value="${radians( 115)}" />
-    <xacro:property name="j3_velocity_limit" value="${radians( 125)}" />
-    <xacro:property name="j4_velocity_limit" value="${radians( 180)}" />
-    <xacro:property name="j5_velocity_limit" value="${radians( 180)}" />
-    <xacro:property name="j6_velocity_limit" value="${radians( 260)}" />
+    <xacro:property name="j1_upper_limit" value="${radians(185)}" />
+    <xacro:property name="j2_upper_limit" value="${radians(76)}" />
+    <xacro:property name="j3_upper_limit" value="${radians(180)}" />
+    <xacro:property name="j4_upper_limit" value="${radians(360)}" />
+    <xacro:property name="j5_upper_limit" value="${radians(125)}" />
+    <xacro:property name="j6_upper_limit" value="${radians(360)}" />
+    <xacro:property name="j1_effort_limit" value="10000" />
+    <xacro:property name="j2_effort_limit" value="20000" />
+    <xacro:property name="j3_effort_limit" value="20000" />
+    <xacro:property name="j4_effort_limit" value="4000" />
+    <xacro:property name="j5_effort_limit" value="4000" />
+    <xacro:property name="j6_effort_limit" value="3000" />
+    <xacro:property name="j1_velocity_limit" value="${radians(130)}" />
+    <xacro:property name="j2_velocity_limit" value="${radians(115)}" />
+    <xacro:property name="j3_velocity_limit" value="${radians(125)}" />
+    <xacro:property name="j4_velocity_limit" value="${radians(180)}" />
+    <xacro:property name="j5_velocity_limit" value="${radians(180)}" />
+    <xacro:property name="j6_velocity_limit" value="${radians(260)}" />
     <!-- links -->
     <link name="${prefix}base_link">
@@ -56,4 +56,16 @@
         </geometry>
       </collision>
+      <inertial>
+        <mass value=" 189" />
+        <origin xyz="-.104 -.00417  .135" />
+        <inertia
+          ixx=" 5.97"
+          ixy=" .0715"
+          ixz="-.13"
+          iyy=" 11.6"
+          iyz=" .00638"
+          izz=" 14.8"
+        />
+      </inertial>
     </link>
     <link name="${prefix}J1_link">
@@ -74,4 +86,16 @@
         </geometry>
       </collision>
+      <inertial>
+        <mass value=" 358" />
+        <origin xyz=" .0206  .0683 -.123" />
+        <inertia
+          ixx=" 18.5"
+          ixy=" 3.57"
+          ixz="-1.4"
+          iyy=" 25.9"
+          iyz="-.486"
+          izz=" 30.2"
+        />
+      </inertial>
     </link>
     <link name="${prefix}J2_link">
@@ -92,4 +116,16 @@
         </geometry>
       </collision>
+      <inertial>
+        <mass value=" 198" />
+        <origin xyz="-.00183  .229  .441" />
+        <inertia
+          ixx=" 26"
+          ixy=" .101"
+          ixz="-.718"
+          iyy=" 26.7"
+          iyz="-1.98"
+          izz=" 3.8"
+        />
+      </inertial>
     </link>
     <link name="${prefix}J3_link">
@@ -110,4 +146,16 @@
         </geometry>
       </collision>
+      <inertial>
+        <mass value=" 340" />
+        <origin xyz=" .485  .0541  .13" />
+        <inertia
+          ixx=" 10.4"
+          ixy=" 2.41"
+          ixz="-5.72"
+          iyy=" 60.3"
+          iyz=" .558"
+          izz=" 61"
+        />
+      </inertial>
     </link>
     <link name="${prefix}J4_link">
@@ -128,4 +176,16 @@
         </geometry>
       </collision>
+      <inertial>
+        <mass value=" 9.92" />
+        <origin xyz=" 1.63 -.00867 -.00000000998" />
+        <inertia
+          ixx=" .0388"
+          ixy=" .00521"
+          ixz="-.00000000746"
+          iyy=" .0892"
+          iyz="-.000000000594"
+          izz=" .0871"
+        />
+      </inertial>
     </link>
     <link name="${prefix}J5_link">
@@ -146,4 +206,16 @@
         </geometry>
       </collision>
+      <inertial>
+        <mass value=" 18" />
+        <origin xyz=" .0485 -.0214  .00000000178" />
+        <inertia
+          ixx=" .134"
+          ixy="-.0205"
+          ixz=" .000000000578"
+          iyy=" .159"
+          iyz=" .00000000843"
+          izz=" .197"
+        />
+      </inertial>
     </link>
     <link name="${prefix}J6_link">
@@ -164,4 +236,16 @@
         </geometry>
       </collision>
+      <inertial>
+        <mass value=" .925" />
+        <origin xyz=" .198  .000000000699  .0000957" />
+        <inertia
+          ixx=" .00259"
+          ixy="-.00000000000463"
+          ixz="-.00000066"
+          iyy=" .00139"
+          iyz=" .0000000000599"
+          izz=" .0014"
+        />
+      </inertial>
     </link>
     <!-- joints -->
@@ -252,4 +336,11 @@
       <child link="${prefix}flange" />
     </joint>
+    <!-- FANUC flange coords -->
+    <link name="${prefix}fanuc_flange" />
+    <joint name="${prefix}flange-fanuc_flange" type="fixed">
+      <origin xyz="0 0 0" rpy="${radians( 180)} ${radians(-90)} ${radians( 0)}" />
+      <parent link="${prefix}flange" />
+      <child link="${prefix}fanuc_flange" />
+    </joint>
     <!-- Attach to parent -->
     <joint name="${prefix}base_joint" type="fixed">
